File: MultiClockDiv/MultiClockDiv_main/MultiClockDiv.sch (KiCad schematic (older format))
At the start: 32 parts, among them J1 GATE OUT1, J2 GATE OUT2, J3 MASTER CLOCK OUT, J4 EXTERNAL CLOCK IN, J5 Conn_01x16_Male, SW1 SW_SPDT

Commit message: correct
Parts:
- removed J5: Conn_01x16_Male, Connector_IDC:IDC-Header_2x08_P2.54mm_Vertical, symbol Connector:Conn_01x16_Male
- added J5: POWER, Connector_IDC:IDC-Header_2x05_P2.54mm_Vertical, symbol MultiClockDiv-rescue:Conn_01x10_Male-Connector
- A1: symbol MCU_Module:Arduino_Nano_v3.x -> MultiClockDiv-rescue:Arduino_Nano_v3.x-MCU_Module
- C1, C2: symbol Device:C -> MultiClockDiv-rescue:C-Device
- D1, D4, D7: symbol Device:LED -> MultiClockDiv-rescue:LED-Device
- D10, D11, D2, D3, D5, D6, D8: symbol Device:D_Schottky -> MultiClockDiv-rescue:D_Schottky-Device
- D9: symbol Device:D -> MultiClockDiv-rescue:D-Device
- J1, J2, J3, J4: symbol Connector:AudioJack2 -> MultiClockDiv-rescue:AudioJack2-Connector
- MULTI/DIV1: renamed from RV1; symbol Device:R_POT -> MultiClockDiv-rescue:R_POT-Device
- R1, R10, R2, R3, R4, R5, R6, R7, R8, R9: symbol Device:R -> MultiClockDiv-rescue:R-Device
- RATE1: renamed from RV2; symbol Device:R_POT -> MultiClockDiv-rescue:R_POT-Device
- SW1: value SW_SPDT -> SELECT; symbol Switch:SW_SPDT -> MultiClockDiv-rescue:SW_SPDT-Switch
Connections:
- net GND: now also J5.3 (Pin_3), J5.4 (Pin_4), J5.5 (Pin_5), J5.6 (Pin_6), J5.7 (Pin_7), J5.8 (Pin_8); no longer D8.2 (A)
- net at A1.6 (D3), D10.2 (A), D11.1 (K)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: no longer D8.1 (K)
- net at R7.2: now also D8.1 (K); no longer D9.1 (K)
- net 12V: no longer names the net of A1.30 (VIN)
- net 12V: now also J5.10 (Pin_10), J5.9 (Pin_9)
- new net: D8.2 (A), D9.1 (K)
- no-connect marks 29 -> 23
Other:
- moved on the sheet: D8, D9
