File: Sampler/sampler_main/sampler.kicad_pcb (KiCad board)
At the start: 2 copper layers, 29 x 99.5 mm, 33 parts, among them J1 TRIG1, J2 TRIG2, J3 OUT, J4 POWER, SW1 ON OFF ON, U1 DFR0299

Commit message: addfile
Other:
- board text added: "Designed by HAGIWO Mar 2021 V.1.0"
