File: MultiClockDiv/panel/panel.kicad_pcb (KiCad board)
At the start: 2 copper layers, 95.7 x 128.5 mm, 44 parts, among them J1 GATE OUT1, J2 GATE OUT2, J3 MASTER CLOCK OUT, J4 EXTERNAL CLOCK IN, J5 Conn_01x16_Male, SW1 SW_SPDT

Commit message: commit
Parts:
- removed A1: Arduino_Nano_v3.x, Module:Arduino_Nano
- removed C1, C2: 220pF, Capacitor_THT:C_Disc_D4.3mm_W1.9mm_P5.00mm
- removed D1, D4, D7: LED, LED_THT:LED_D3.0mm
- removed D10, D11, D2, D3, D5, D6, D8: BAT43, Diode_THT:D_DO-41_SOD81_P10.16mm_Horizontal
- removed D9: D, Diode_THT:D_DO-41_SOD81_P10.16mm_Horizontal
- removed J1: GATE OUT1, Connector_Audio:Jack_3.5mm_QingPu_WQP-PJ398SM_Vertical_CircularHoles
- removed J2: GATE OUT2, Connector_Audio:Jack_3.5mm_QingPu_WQP-PJ398SM_Vertical_CircularHoles
- removed J3: MASTER CLOCK OUT, Connector_Audio:Jack_3.5mm_QingPu_WQP-PJ398SM_Vertical_CircularHoles
- removed J4: EXTERNAL CLOCK IN, Connector_Audio:Jack_3.5mm_QingPu_WQP-PJ398SM_Vertical_CircularHoles
- removed J5: Conn_01x16_Male, Connector_IDC:IDC-Header_2x08_P2.54mm_Vertical
- removed R1, R2, R3, R5, R7, R8: 470R, Resistor_THT:R_Axial_DIN0207_L6.3mm_D2.5mm_P7.62mm_Horizontal
- removed R10, R4, R6, R9: 22K, Resistor_THT:R_Axial_DIN0207_L6.3mm_D2.5mm_P7.62mm_Horizontal
- removed RV1, RV2: 100K, Potentiometer_THT:Potentiometer_Alps_RK09K_Single_Vertical
- removed SW1: SW_SPDT, digikey-footprints:Toggle_Switch_100SP1T1B4M2QE
- added H10: SLIDE, elektrophon:panel_potentiometer, F.Cu at (36.9, 136.8)
- added H10: SLIDE, elektrophon:panel_potentiometer, F.Cu at (37.0, 121.5)
- moved H4 16.4 mm to (53.6, 136.7)
- moved H9 12.5 mm to (53.6, 121.8)
- moved H3 11.2 mm to (53.6, 106.9)
- moved H1 6.64 mm to (37.1, 106.8)
- moved H2 2.35 mm to (41.3, 93.9)
- moved H10 2.29 mm to (51.7, 94.1)
- moved H11 0.10 mm to (45.7, 69.3)
Other:
- board size 95.7 x 128.5 mm -> 40.6 x 128.5 mm
- board text removed: "Designed by HAGIWO Mar 2021 V.1.0"

Commit message: first commit
Parts:
- added G***: LOGO, logo:silk8, F.Cu at (47.9, 89.3)

Commit message: correct
Parts:
- removed the G*** at (47.9, 89.3)
- added G***: LOGO, logo:silk13, F.Cu at (46.6, 89.3)
- H1: value SLIDE -> IN
- H12: value SCALE -> RATE
- H2: value ON/EXT -> CH1/CH2
- H3: value TRIG -> OUT
- H4: value CV IN -> CH2
- H9: value CV -> CH1
- moved H11 3.60 mm to (45.7, 72.9)
- moved H2 2.55 mm to (38.8, 93.9)
- moved H10 2.02 mm to (53.7, 94.0)

Commit message: correct
Parts:
- removed G***: LOGO, logo:silk13
- removed the H5 at (58.3, 153.3)
- removed the H5 at (58.4, 30.9)
- added ?: , , F.Cu at (93.3, 88.0)
- added ?: , , F.Cu at (87.4, 45.5)
- added ?: , , F.Cu at (107.0, 60.9)
- added H5: MountingHole, MountingHole:MountingHole_3.2mm_M3, F.Cu at (28.8, 142.7)
- added H5: MountingHole, MountingHole:MountingHole_3.2mm_M3, F.Cu at (48.2, 153.3)
- moved H6 110.2 mm to (52.0, 44.8)
- moved H12 7.40 mm to (40.8, 45.1)
- moved H3 6.25 mm to (47.4, 106.9)
- moved H4 6.25 mm to (47.4, 136.7)
- moved H9 6.25 mm to (47.4, 121.8)
- moved H10 6.22 mm to (47.5, 94.0)
- moved H2 5.25 mm to (33.5, 93.9)
- moved H11 5.10 mm to (40.8, 71.5)
- moved H1 3.75 mm to (33.4, 106.8)
- moved H10 3.75 mm to (33.1, 136.8)
- moved H10 3.75 mm to (33.2, 121.5)
Other:
- board size 40.6 x 128.5 mm -> 30.5 x 128.5 mm

Commit message: addPanel
Parts:
- added G***: LOGO, LOGO:silk22, F.Cu at (41.4, 88.7)
Other:
- board text added: "HAGIWO"
