File: Quantizer/panel/panel.kicad_pcb (KiCad board)
At the start: 2 copper layers, 50.8 x 128.5 mm, 13 parts

Commit message: First commit
Parts:
- moved H5 0.30 mm to (68.5, 153.3)

Commit message: correct
Parts:
- removed the H5 at (68.5, 30.9)
- removed H6: MountingHole, MountingHole:MountingHole_3.2mm_M3
Other:
- board outline removed

Commit message: correct
Parts:
- moved G*** 47.7 mm to (98.8, 93.9)
- moved H1 47.7 mm to (85.6, 121.2)
- moved H10 47.7 mm to (97.8, 102.5)
- moved H11 47.7 mm to (97.8, 78.4)
- moved H12 47.7 mm to (97.8, 56.5)
- moved H3 47.7 mm to (109.9, 121.2)
- moved H4 47.7 mm to (85.6, 138.2)
- moved H5 47.7 mm to (115.6, 161.2)
- moved H5 47.7 mm to (79.8, 38.7)
- moved H9 47.7 mm to (109.9, 138.3)
- moved H2 47.7 mm to (97.8, 91.2)
Other:
- board outline added: 30.5 x 128.5 mm
