File: CHORD_VCO/CHORD_VCO.sch (KiCad schematic (older format))
At the start: 40 parts, among them J1 1V/OCT, J2 INVERSION_CV, J3 CHORD_CV, J4 OUT, J5 POWER, U1 MCP6L02x-xSN

Commit message: AddPCB
Parts:
- J1, J2, J3, J4: footprint (none) -> Connector_Audio:Jack_3.5mm_QingPu_WQP-PJ398SM_Vertical_CircularHoles
- J5: footprint (none) -> Connector_IDC:IDC-Header_2x05_P2.54mm_Vertical
Changed lines of the file:
@@
 F 0 "J1" H 1371 2333 50  0000 R CNN
 F 1 "1V/OCT" H 1371 2424 50  0000 R CNN
-F 2 "" H 1550 2350 50  0001 C CNN
+F 2 "Connector_Audio:Jack_3.5mm_QingPu_WQP-PJ398SM_Vertical_CircularHoles" H 1550 2350 50  0001 C CNN
 F 3 "~" H 1550 2350 50  0001 C CNN
 	1    1550 2350
@@
 F 0 "J2" H 5820 2333 50  0000 R CNN
 F 1 "INVERSION_CV" H 5820 2424 50  0000 R CNN
-F 2 "" H 6000 2350 50  0001 C CNN
+F 2 "Connector_Audio:Jack_3.5mm_QingPu_WQP-PJ398SM_Vertical_CircularHoles" H 6000 2350 50  0001 C CNN
 F 3 "~" H 6000 2350 50  0001 C CNN
 	1    6000 2350
@@
 F 0 "J3" H 5820 3633 50  0000 R CNN
 F 1 "CHORD_CV" H 5820 3724 50  0000 R CNN
-F 2 "" H 6000 3650 50  0001 C CNN
+F 2 "Connector_Audio:Jack_3.5mm_QingPu_WQP-PJ398SM_Vertical_CircularHoles" H 6000 3650 50  0001 C CNN
 F 3 "~" H 6000 3650 50  0001 C CNN
 	1    6000 3650
@@
 F 0 "J4" H 7770 5283 50  0000 R CNN
 F 1 "OUT" H 7770 5374 50  0000 R CNN
-F 2 "" H 7950 5300 50  0001 C CNN
+F 2 "Connector_Audio:Jack_3.5mm_QingPu_WQP-PJ398SM_Vertical_CircularHoles" H 7950 5300 50  0001 C CNN
 F 3 "~" H 7950 5300 50  0001 C CNN
 	1    7950 5300
@@
 F 0 "J5" H 9108 5931 50  0000 C CNN
 F 1 "POWER" H 9108 5840 50  0000 C CNN
-F 2 "" H 9000 5350 50  0001 C CNN
+F 2 "Connector_IDC:IDC-Header_2x05_P2.54mm_Vertical" H 9000 5350 50  0001 C CNN
 F 3 "~" H 9000 5350 50  0001 C CNN
 	1    9000 5350
